File: 1s_lipo.kicad_sch (KiCad schematic)
At the start: 18 parts, among them J3 LiPo 1S, U4 DW01, U5 AP2112K-3.3, U6 PM8205A, U7 HX4054A

Commit message: gregdavill: Initial commit of new badge design
Parts:
- removed U5: AP2112K-3.3, Package_TO_SOT_SMD:SOT-23-5, symbol Regulator_Linear:AP2112K-3.3
- added C13, C14: 10uF, Capacitor_SMD:C_0603_1608Metric, symbol Device:C
- added L1: 2.2uH, Inductor_SMD:L_0805_2012Metric, symbol Device:L_Small
- added R17: 360k, Resistor_SMD:R_0603_1608Metric, symbol Device:R
- added R18: 82k, Resistor_SMD:R_0603_1608Metric, symbol Device:R
- added U7: TLV62569DBV, Package_TO_SOT_SMD:SOT-23-5, symbol Regulator_Switching:TLV62569DBV
- C10: value 1uF -> 10pF; Mfg (none) -> Samsung Electro-Mechanics; Mfg_1 (none) -> YAGEO; PN (none) -> CL03C100JA3GNNC; PN_1 (none) -> CC0201DRNPO8BN100
- C9: value 1uF -> 10uF; Mfg (none) -> Murata Electronics North America; Mfg_1 (none) -> YAGEO; PN (none) -> GRM155R60J106ME15D; PN_1 (none) -> CC0402MRX5R5BB106
- renumbered D26 to D514, R12 to R10, R13 to R11, R14 to R12, R15 to R13, R16 to R14, R17 to R15, R18 to R16, U4 to U6, U6 to U8, U7 to U9
Connections:
- net BATT_PLUS: now also C9.2, U7.1 (EN), U7.4 (VIN); no longer C9.1
- net GND: now also C9.1, C13.1, C14.1, R18.2, U7.2 (GND); no longer C10.2, C9.2
- net VCC: now also C10.2, C13.2, C14.2, L1.2, R17.2; no longer C10.1
- new net: C10.1, R17.1, R18.1, U7.5 (FB)
- new net: L1.1, U7.3 (SW)
Other:
- note added: "3.3V @ 1A - System IO"
