File: 1s_lipo.kicad_sch (KiCad schematic)
At the start: 23 parts, among them J3 LiPo 1S, U6 DW01, U7 TLV62569DBV, U8 PM8205A, U9 HX4054A

Commit message: add BOM
Parts:
- C10: Mfg_1 YAGEO -> (none); PN CL03C100JA3GNNC -> CL10C100JB81PNC; PN_1 CC0201DRNPO8BN100 -> (none)
- C11, C8: Mfg (none) -> Samsung Electro-Mechanics; PN (none) -> CL10B104KB8NNNC
- C12: Mfg (none) -> Samsung Electro-Mechanics; PN (none) -> CL10A475KO8NNNC
- C13, C14, C9: Mfg Murata Electronics North America -> Samsung Electro-Mechanics; Mfg_1 YAGEO -> (none); PN GRM155R60J106ME15D -> CL10A106MO8NQNC; PN_1 CC0402MRX5R5BB106 -> (none)
- D514: Mfg (none) -> Foshan NationStar Optoelectronics; PN (none) -> NCD0603Y1
- J3: Mfg (none) -> JST Sales America; PN (none) -> S2B-PH-SM4-TB(LF)(SN)
- L1: Mfg Murata Electronics -> Sunltech Tech; Mfg_1 Sunltech Tech -> (none); PN LQM21PN2R2NGCD -> SLM20122R2MIT; PN_1 SLM20122R2MIT -> (none)
- R10: Mfg (none) -> UNI-ROYAL(Uniroyal Elec); PN (none) -> 0603WAF1000T5E
- R11, R15: Mfg (none) -> UNI-ROYAL(Uniroyal Elec); PN (none) -> 0603WAF1001T5E
- R12, R13, R14: Mfg (none) -> UNI-ROYAL(Uniroyal Elec); PN (none) -> 0603WAF0000T5E
- R16: Mfg (none) -> UNI-ROYAL(Uniroyal Elec); PN (none) -> 0603WAF2001T5E
- R17: Mfg ‎Yageo‎ -> UNI-ROYAL(Uniroyal Elec); Mfg_1 UNI-ROYAL(Uniroyal Elec) -> (none); PN RC0201FR-07360KL -> 0603WAF3603T5E; PN_1 0201WMF3603TCE -> (none)
- R18: Mfg ‎Yageo‎ -> UNI-ROYAL(Uniroyal Elec); Mfg_1 UNI-ROYAL(Uniroyal Elec) -> (none); PN RC0201FR-0782KL -> 0603WAF8202T5E; PN_1 0201WMF8202TCE -> (none)
- U6: Mfg (none) -> Guangdong Hottech; PN (none) -> DW01
- U7: Mfg (none) -> Texas Instruments; PN (none) -> TLV62569DBVR
- U8: Mfg (none) -> PN SILICON; PN (none) -> PM8205A
- U9: Mfg (none) -> HX(hengjiaxing); PN (none) -> HX4054A
