File: badge.kicad_pcb (KiCad board)
At the start: 2 copper layers, 100 x 100 mm, 3 parts

Commit message: Added schematic, board and gerbers for my fork
Signed-off-by: Thomas Flummer <tf@flummer.net>
Parts:
- added C1: 1uF, Capacitor_SMD:C_0603_1608Metric, F.Cu at (81.9, 101.5)
- added C10: 1uF, Capacitor_SMD:C_0603_1608Metric, F.Cu at (63.0, 134.2)
- added C11: 100nF, Capacitor_SMD:C_0603_1608Metric, F.Cu at (62.6, 120.2)
- added C12: 4.7uF, Capacitor_SMD:C_0603_1608Metric, F.Cu at (69.2, 119.3)
- added C2: 100nF, Capacitor_SMD:C_0603_1608Metric, F.Cu at (83.5, 101.5)
- added C3: 1uF, Capacitor_SMD:C_0603_1608Metric, F.Cu at (98.6, 116.4)
- added C4: 100nF, Capacitor_SMD:C_0603_1608Metric, F.Cu at (98.6, 114.8)
- added C5: 1uF, Capacitor_SMD:C_0603_1608Metric, F.Cu at (80.8, 126.3)
- added C6: 100nF, Capacitor_SMD:C_0603_1608Metric, F.Cu at (66.3, 125.2)
- added C7: 10uF, Capacitor_SMD:C_0603_1608Metric, F.Cu at (74.2, 118.8)
- added C8: 100nF, Capacitor_SMD:C_0603_1608Metric, F.Cu at (68.8, 109.1)
- added C9: 1uF, Capacitor_SMD:C_0603_1608Metric, F.Cu at (63.0, 128.6)
- added D1: LED_ARGB, Opto:ARGB-1x1mm, F.Cu at (103.7, 53.9)
- added D10: LED_ARGB, Opto:ARGB-1x1mm, F.Cu at (81.8, 81.8)
- added D11: LED_ARGB, Opto:ARGB-1x1mm, F.Cu at (78.9, 84.5)
- added D12: LED_ARGB, Opto:ARGB-1x1mm, F.Cu at (76.0, 87.2)
- added D13: LED_ARGB, Opto:ARGB-1x1mm, F.Cu at (112.8, 124.0)
- added D14: LED_ARGB, Opto:ARGB-1x1mm, F.Cu at (115.5, 121.1)
- added D15: LED_ARGB, Opto:ARGB-1x1mm, F.Cu at (118.2, 118.2)
- added D16: LED_ARGB, Opto:ARGB-1x1mm, F.Cu at (121.1, 115.5)
- added D17: LED_ARGB, Opto:ARGB-1x1mm, F.Cu at (124.0, 112.8)
- added D18: LED_ARGB, Opto:ARGB-1x1mm, F.Cu at (126.9, 110.2)
- added D19: LED_ARGB, Opto:ARGB-1x1mm, F.Cu at (130.0, 107.7)
- added D2: LED_ARGB, Opto:ARGB-1x1mm, F.Cu at (101.6, 57.2)
- added D20: LED_ARGB, Opto:ARGB-1x1mm, F.Cu at (133.1, 105.2)
- added D21: LED_ARGB, Opto:ARGB-1x1mm, F.Cu at (136.2, 102.8)
- added D22: LED_ARGB, Opto:ARGB-1x1mm, F.Cu at (139.5, 100.6)
- added D23: LED_ARGB, Opto:ARGB-1x1mm, F.Cu at (142.8, 98.4)
- added D24: LED_ARGB, Opto:ARGB-1x1mm, F.Cu at (146.1, 96.3)
- added D25: LED, LED_SMD:LED_0603_1608Metric, F.Cu at (80.7, 119.3)
- added D26: CHRG, LED_SMD:LED_0603_1608Metric, F.Cu at (61.9, 122.7)
- added D3: LED_ARGB, Opto:ARGB-1x1mm, F.Cu at (99.4, 60.5)
- added D4: LED_ARGB, Opto:ARGB-1x1mm, F.Cu at (97.2, 63.8)
- added D5: LED_ARGB, Opto:ARGB-1x1mm, F.Cu at (94.8, 66.9)
- added D6: LED_ARGB, Opto:ARGB-1x1mm, F.Cu at (92.3, 70.0)
- added D7: LED_ARGB, Opto:ARGB-1x1mm, F.Cu at (89.8, 73.1)
- added D8: LED_ARGB, Opto:ARGB-1x1mm, F.Cu at (87.2, 76.0)
- added D9: LED_ARGB, Opto:ARGB-1x1mm, F.Cu at (84.5, 78.9)
- added G***: LOGO, Aesthetics:kicon_2020_name_silk, F.Cu at (56.1, 125.8)
- added IC1: SAMD21G18A-MU, Package_DFN_QFN:QFN-48-1EP_7x7mm_P0.5mm_EP5.3x5.3mm, F.Cu at (74.0, 126.0)
- added J1: USB_C, Connectors:USB_C_Receptacle_U262-161N-4BVC11, F.Cu at (70.7, 145.6)
- added J2: DEBUG, Connector_PinHeader_2.54mm:PinHeader_1x06_P2.54mm_Vertical, B.Cu at (81.0, 146.0)
- added J3: LiPo 1S, Connectors:PH2.0-SMD-Horizontal, B.Cu at (58.0, 113.0)
- added R10: 4.7k, Resistor_SMD:R_0603_1608Metric, F.Cu at (90.6, 110.5)
- added R11: 100k, Resistor_SMD:R_0603_1608Metric, F.Cu at (80.8, 129.8)
- added R12: 100, Resistor_SMD:R_0603_1608Metric, F.Cu at (62.6, 109.1)
- added R13: 1k, Resistor_SMD:R_0603_1608Metric, F.Cu at (65.7, 109.1)
- added R14: 1, Resistor_SMD:R_0603_1608Metric, F.Cu at (66.8, 115.7)
- added R15: 1, Resistor_SMD:R_0603_1608Metric, F.Cu at (65.2, 115.7)
- added R16: 1, Resistor_SMD:R_0603_1608Metric, F.Cu at (62.6, 118.4)
- added R17: 1k, Resistor_SMD:R_0603_1608Metric, F.Cu at (61.9, 126.0)
- added R18: 2k, Resistor_SMD:R_0603_1608Metric, F.Cu at (66.2, 122.1)
- added R2: 3k3, Resistor_SMD:R_0603_1608Metric, F.Cu at (85.0, 101.5)
- added R4: 3k3, Resistor_SMD:R_0603_1608Metric, F.Cu at (98.6, 118.0)
- added R5: 5.1k, Resistor_SMD:R_0603_1608Metric, F.Cu at (68.4, 137.5)
- added R6: 5.1k, Resistor_SMD:R_0603_1608Metric, F.Cu at (73.2, 137.6)
- added R7: 10k, Resistor_SMD:R_0603_1608Metric, F.Cu at (81.9, 121.5)
- added R8: 1k, Resistor_SMD:R_0603_1608Metric, F.Cu at (78.4, 118.1)
- added R9: 4.7k, Resistor_SMD:R_0603_1608Metric, F.Cu at (89.4, 109.3)
- added REF**: Small_SMD_Proto_Pad, Connectors:Small_SMD_Proto_Pad, F.Cu at (110.8, 100.6)
- added REF**: Small_SMD_Proto_Pad, Connectors:Small_SMD_Proto_Pad, F.Cu at (103.2, 91.7)
- added REF**: PTH_Proto_pad, Connectors:PTH_Proto_pad, F.Cu at (107.6, 88.6)
- added REF**: Small_SMD_Proto_Pad, Connectors:Small_SMD_Proto_Pad, B.Cu at (112.1, 100.6)
- added REF**: Small_SMD_Proto_Pad, Connectors:Small_SMD_Proto_Pad, B.Cu at (107.0, 76.5)
- added REF**: Small_SMD_Proto_Pad, Connectors:Small_SMD_Proto_Pad, B.Cu at (104.4, 75.2)
- added REF**: Small_SMD_Proto_Pad, Connectors:Small_SMD_Proto_Pad, B.Cu at (126.0, 89.2)
- added REF**: Small_SMD_Proto_Pad, Connectors:Small_SMD_Proto_Pad, B.Cu at (110.8, 63.8)
- added REF**: Small_SMD_Proto_Pad, Connectors:Small_SMD_Proto_Pad, B.Cu at (113.3, 86.7)
- added REF**: Small_SMD_Proto_Pad, Connectors:Small_SMD_Proto_Pad, B.Cu at (98.1, 93.0)
- added REF**: Small_SMD_Proto_Pad, Connectors:Small_SMD_Proto_Pad, B.Cu at (142.5, 89.2)
- added REF**: Small_SMD_Proto_Pad, Connectors:Small_SMD_Proto_Pad, B.Cu at (108.3, 108.3)
- added REF**: Small_SMD_Proto_Pad, Connectors:Small_SMD_Proto_Pad, B.Cu at (99.4, 74.0)
- added REF**: Small_SMD_Proto_Pad, Connectors:Small_SMD_Proto_Pad, F.Cu at (96.8, 94.3)
- added REF**: Small_SMD_Proto_Pad, Connectors:Small_SMD_Proto_Pad, B.Cu at (117.1, 99.4)
- added REF**: Small_SMD_Proto_Pad, Connectors:Small_SMD_Proto_Pad, B.Cu at (119.7, 96.8)
- added REF**: Small_SMD_Proto_Pad, Connectors:Small_SMD_Proto_Pad, B.Cu at (108.3, 65.1)
- added REF**: Small_SMD_Proto_Pad, Connectors:Small_SMD_Proto_Pad, B.Cu at (107.0, 62.5)
- added REF**: Small_SMD_Proto_Pad, Connectors:Small_SMD_Proto_Pad, B.Cu at (107.0, 99.4)
- added REF**: Small_SMD_Proto_Pad, Connectors:Small_SMD_Proto_Pad, B.Cu at (93.0, 91.7)
- added REF**: Small_SMD_Proto_Pad, Connectors:Small_SMD_Proto_Pad, B.Cu at (115.9, 86.7)
- added REF**: Small_SMD_Proto_Pad, Connectors:Small_SMD_Proto_Pad, B.Cu at (108.3, 101.9)
- added REF**: Small_SMD_Proto_Pad, Connectors:Small_SMD_Proto_Pad, B.Cu at (129.8, 90.5)
- added REF**: Small_SMD_Proto_Pad, Connectors:Small_SMD_Proto_Pad, B.Cu at (138.7, 86.7)
- added REF**: Small_SMD_Proto_Pad, Connectors:Small_SMD_Proto_Pad, F.Cu at (118.4, 79.0)
- added REF**: Small_SMD_Proto_Pad, Connectors:Small_SMD_Proto_Pad, B.Cu at (123.5, 105.7)
- added REF**: Small_SMD_Proto_Pad, Connectors:Small_SMD_Proto_Pad, B.Cu at (113.3, 72.7)
- added REF**: Small_SMD_Proto_Pad, Connectors:Small_SMD_Proto_Pad, B.Cu at (113.3, 98.1)
- added REF**: Small_SMD_Proto_Pad, Connectors:Small_SMD_Proto_Pad, B.Cu at (100.6, 68.9)
- added REF**: Small_SMD_Proto_Pad, Connectors:Small_SMD_Proto_Pad, B.Cu at (104.4, 71.4)
- added REF**: Small_SMD_Proto_Pad, Connectors:Small_SMD_Proto_Pad, B.Cu at (112.1, 68.9)
- added REF**: Small_SMD_Proto_Pad, Connectors:Small_SMD_Proto_Pad, B.Cu at (124.8, 86.7)
- added REF**: Small_SMD_Proto_Pad, Connectors:Small_SMD_Proto_Pad, B.Cu at (87.9, 80.3)
- added REF**: Small_SMD_Proto_Pad, Connectors:Small_SMD_Proto_Pad, B.Cu at (129.8, 98.1)
- added REF**: Small_SMD_Proto_Pad, Connectors:Small_SMD_Proto_Pad, B.Cu at (133.7, 93.0)
- added REF**: PTH_Proto_pad, Connectors:PTH_Proto_pad, F.Cu at (110.2, 81.0)
- added REF**: Small_SMD_Proto_Pad, Connectors:Small_SMD_Proto_Pad, B.Cu at (101.9, 80.3)
- added REF**: Small_SMD_Proto_Pad, Connectors:Small_SMD_Proto_Pad, B.Cu at (110.8, 90.5)
- added REF**: Small_SMD_Proto_Pad, Connectors:Small_SMD_Proto_Pad, B.Cu at (113.3, 84.1)
- added REF**: Small_SMD_Proto_Pad, Connectors:Small_SMD_Proto_Pad, B.Cu at (93.0, 85.4)
- added REF**: Small_SMD_Proto_Pad, Connectors:Small_SMD_Proto_Pad, B.Cu at (119.7, 86.7)
- added REF**: Small_SMD_Proto_Pad, Connectors:Small_SMD_Proto_Pad, B.Cu at (95.6, 80.3)
- added REF**: Small_SMD_Proto_Pad, Connectors:Small_SMD_Proto_Pad, B.Cu at (117.1, 104.4)
- added REF**: Small_SMD_Proto_Pad, Connectors:Small_SMD_Proto_Pad, B.Cu at (121.0, 99.4)
- added REF**: Small_SMD_Proto_Pad, Connectors:Small_SMD_Proto_Pad, B.Cu at (122.2, 86.7)
- added REF**: Small_SMD_Proto_Pad, Connectors:Small_SMD_Proto_Pad, B.Cu at (105.7, 68.9)
- added REF**: Small_SMD_Proto_Pad, Connectors:Small_SMD_Proto_Pad, F.Cu at (101.9, 98.1)
- added REF**: Small_SMD_Proto_Pad, Connectors:Small_SMD_Proto_Pad, B.Cu at (110.8, 95.6)
- added REF**: Small_SMD_Proto_Pad, Connectors:Small_SMD_Proto_Pad, B.Cu at (98.1, 89.2)
- added REF**: Small_SMD_Proto_Pad, Connectors:Small_SMD_Proto_Pad, B.Cu at (115.9, 98.1)
- added REF**: Small_SMD_Proto_Pad, Connectors:Small_SMD_Proto_Pad, B.Cu at (104.4, 76.5)
- added REF**: Small_SMD_Proto_Pad, Connectors:Small_SMD_Proto_Pad, B.Cu at (132.4, 90.5)
- added REF**: Small_SMD_Proto_Pad, Connectors:Small_SMD_Proto_Pad, B.Cu at (121.0, 95.6)
- added REF**: Small_SMD_Proto_Pad, Connectors:Small_SMD_Proto_Pad, B.Cu at (137.5, 87.9)
- added REF**: Small_SMD_Proto_Pad, Connectors:Small_SMD_Proto_Pad, B.Cu at (114.6, 96.8)
- added REF**: Small_SMD_Proto_Pad, Connectors:Small_SMD_Proto_Pad, B.Cu at (103.2, 98.1)
- added REF**: Small_SMD_Proto_Pad, Connectors:Small_SMD_Proto_Pad, B.Cu at (108.3, 63.8)
- added REF**: Small_SMD_Proto_Pad, Connectors:Small_SMD_Proto_Pad, F.Cu at (124.8, 93.0)
- added REF**: Small_SMD_Proto_Pad, Connectors:Small_SMD_Proto_Pad, B.Cu at (107.0, 63.8)
- added REF**: Small_SMD_Proto_Pad, Connectors:Small_SMD_Proto_Pad, B.Cu at (128.6, 87.9)
- added REF**: Small_SMD_Proto_Pad, Connectors:Small_SMD_Proto_Pad, B.Cu at (98.1, 90.5)
- added REF**: Small_SMD_Proto_Pad, Connectors:Small_SMD_Proto_Pad, B.Cu at (108.3, 104.4)
- added REF**: Small_SMD_Proto_Pad, Connectors:Small_SMD_Proto_Pad, B.Cu at (110.8, 71.4)
- added REF**: Small_SMD_Proto_Pad, Connectors:Small_SMD_Proto_Pad, B.Cu at (87.9, 85.4)
- added REF**: Small_SMD_Proto_Pad, Connectors:Small_SMD_Proto_Pad, B.Cu at (96.8, 77.8)
- added REF**: Small_SMD_Proto_Pad, Connectors:Small_SMD_Proto_Pad, B.Cu at (137.5, 86.7)
- added REF**: Small_SMD_Proto_Pad, Connectors:Small_SMD_Proto_Pad, B.Cu at (105.7, 98.1)
- added REF**: Small_SMD_Proto_Pad, Connectors:Small_SMD_Proto_Pad, B.Cu at (118.4, 76.5)
- added REF**: Small_SMD_Proto_Pad, Connectors:Small_SMD_Proto_Pad, F.Cu at (114.6, 98.1)
- added REF**: Small_SMD_Proto_Pad, Connectors:Small_SMD_Proto_Pad, B.Cu at (98.1, 87.9)
- added REF**: Small_SMD_Proto_Pad, Connectors:Small_SMD_Proto_Pad, B.Cu at (94.3, 86.7)
- added REF**: Small_SMD_Proto_Pad, Connectors:Small_SMD_Proto_Pad, B.Cu at (105.7, 70.2)
- added REF**: Small_SMD_Proto_Pad, Connectors:Small_SMD_Proto_Pad, B.Cu at (99.4, 87.9)
- added REF**: Small_SMD_Proto_Pad, Connectors:Small_SMD_Proto_Pad, B.Cu at (114.6, 67.6)
- added REF**: Small_SMD_Proto_Pad, Connectors:Small_SMD_Proto_Pad, B.Cu at (89.2, 87.9)
- added REF**: Small_SMD_Proto_Pad, Connectors:Small_SMD_Proto_Pad, B.Cu at (131.1, 94.3)
- added REF**: Small_SMD_Proto_Pad, Connectors:Small_SMD_Proto_Pad, B.Cu at (94.3, 82.9)
- added REF**: Small_SMD_Proto_Pad, Connectors:Small_SMD_Proto_Pad, B.Cu at (138.7, 93.0)
- added REF**: Small_SMD_Proto_Pad, Connectors:Small_SMD_Proto_Pad, B.Cu at (107.0, 67.6)
- added REF**: Small_SMD_Proto_Pad, Connectors:Small_SMD_Proto_Pad, F.Cu at (114.6, 89.2)
- added REF**: Small_SMD_Proto_Pad, Connectors:Small_SMD_Proto_Pad, B.Cu at (131.1, 95.6)
- added REF**: Small_SMD_Proto_Pad, Connectors:Small_SMD_Proto_Pad, B.Cu at (104.4, 66.3)
- added REF**: Small_SMD_Proto_Pad, Connectors:Small_SMD_Proto_Pad, B.Cu at (119.7, 87.9)
- added REF**: Small_SMD_Proto_Pad, Connectors:Small_SMD_Proto_Pad, B.Cu at (99.4, 77.8)
- added REF**: Small_SMD_Proto_Pad, Connectors:Small_SMD_Proto_Pad, B.Cu at (100.6, 77.8)
- added REF**: Small_SMD_Proto_Pad, Connectors:Small_SMD_Proto_Pad, B.Cu at (115.9, 110.8)
- added REF**: Small_SMD_Proto_Pad, Connectors:Small_SMD_Proto_Pad, B.Cu at (133.7, 94.3)
- added REF**: Small_SMD_Proto_Pad, Connectors:Small_SMD_Proto_Pad, B.Cu at (91.7, 91.7)
- added REF**: Small_SMD_Proto_Pad, Connectors:Small_SMD_Proto_Pad, B.Cu at (93.0, 84.1)
- added REF**: Small_SMD_Proto_Pad, Connectors:Small_SMD_Proto_Pad, B.Cu at (132.4, 96.8)
- added REF**: Small_SMD_Proto_Pad, Connectors:Small_SMD_Proto_Pad, F.Cu at (128.6, 93.0)
- added REF**: Small_SMD_Proto_Pad, Connectors:Small_SMD_Proto_Pad, B.Cu at (96.8, 84.1)
- added REF**: Small_SMD_Proto_Pad, Connectors:Small_SMD_Proto_Pad, B.Cu at (90.5, 84.1)
- added REF**: Small_SMD_Proto_Pad, Connectors:Small_SMD_Proto_Pad, B.Cu at (132.4, 91.7)
- added REF**: Small_SMD_Proto_Pad, Connectors:Small_SMD_Proto_Pad, B.Cu at (122.2, 105.7)
- added REF**: Small_SMD_Proto_Pad, Connectors:Small_SMD_Proto_Pad, B.Cu at (119.7, 105.7)
- added REF**: Small_SMD_Proto_Pad, Connectors:Small_SMD_Proto_Pad, B.Cu at (119.7, 98.1)
- added REF**: Small_SMD_Proto_Pad, Connectors:Small_SMD_Proto_Pad, B.Cu at (126.0, 96.8)
- added REF**: Small_SMD_Proto_Pad, Connectors:Small_SMD_Proto_Pad, B.Cu at (94.3, 80.3)
- added REF**: Small_SMD_Proto_Pad, Connectors:Small_SMD_Proto_Pad, B.Cu at (134.9, 95.6)
- added REF**: Small_SMD_Proto_Pad, Connectors:Small_SMD_Proto_Pad, B.Cu at (103.2, 80.3)
- added REF**: Small_SMD_Proto_Pad, Connectors:Small_SMD_Proto_Pad, F.Cu at (103.2, 80.3)
- added REF**: Small_SMD_Proto_Pad, Connectors:Small_SMD_Proto_Pad, B.Cu at (101.9, 101.9)
- added REF**: Small_SMD_Proto_Pad, Connectors:Small_SMD_Proto_Pad, B.Cu at (99.4, 99.4)
- added REF**: Small_SMD_Proto_Pad, Connectors:Small_SMD_Proto_Pad, B.Cu at (86.7, 85.4)
- added REF**: Small_SMD_Proto_Pad, Connectors:Small_SMD_Proto_Pad, B.Cu at (104.4, 68.9)
- added REF**: Small_SMD_Proto_Pad, Connectors:Small_SMD_Proto_Pad, B.Cu at (95.6, 74.0)
- added REF**: Small_SMD_Proto_Pad, Connectors:Small_SMD_Proto_Pad, B.Cu at (122.2, 80.3)
- added REF**: Small_SMD_Proto_Pad, Connectors:Small_SMD_Proto_Pad, B.Cu at (95.6, 77.8)
- added REF**: Small_SMD_Proto_Pad, Connectors:Small_SMD_Proto_Pad, B.Cu at (99.4, 94.3)
- added REF**: Small_SMD_Proto_Pad, Connectors:Small_SMD_Proto_Pad, B.Cu at (95.6, 75.2)
- added REF**: Small_SMD_Proto_Pad, Connectors:Small_SMD_Proto_Pad, B.Cu at (113.3, 70.2)
- added REF**: Small_SMD_Proto_Pad, Connectors:Small_SMD_Proto_Pad, F.Cu at (118.4, 84.1)
- added REF**: Small_SMD_Proto_Pad, Connectors:Small_SMD_Proto_Pad, F.Cu at (109.5, 87.9)
- added REF**: Small_SMD_Proto_Pad, Connectors:Small_SMD_Proto_Pad, B.Cu at (117.1, 82.9)
- added REF**: Small_SMD_Proto_Pad, Connectors:Small_SMD_Proto_Pad, B.Cu at (101.9, 90.5)
- added REF**: Small_SMD_Proto_Pad, Connectors:Small_SMD_Proto_Pad, B.Cu at (137.5, 91.7)
- added REF**: Small_SMD_Proto_Pad, Connectors:Small_SMD_Proto_Pad, B.Cu at (108.3, 74.0)
- added REF**: Small_SMD_Proto_Pad, Connectors:Small_SMD_Proto_Pad, B.Cu at (129.8, 96.8)
- added REF**: Small_SMD_Proto_Pad, Connectors:Small_SMD_Proto_Pad, B.Cu at (109.5, 61.3)
- added REF**: Small_SMD_Proto_Pad, Connectors:Small_SMD_Proto_Pad, B.Cu at (96.8, 96.8)
- added REF**: Small_SMD_Proto_Pad, Connectors:Small_SMD_Proto_Pad, B.Cu at (104.4, 100.6)
- added REF**: Small_SMD_Proto_Pad, Connectors:Small_SMD_Proto_Pad, B.Cu at (110.8, 65.1)
- added REF**: Small_SMD_Proto_Pad, Connectors:Small_SMD_Proto_Pad, B.Cu at (115.9, 84.1)
- added REF**: Small_SMD_Proto_Pad, Connectors:Small_SMD_Proto_Pad, F.Cu at (112.1, 95.6)
- added REF**: Small_SMD_Proto_Pad, Connectors:Small_SMD_Proto_Pad, B.Cu at (114.6, 84.1)
- added REF**: Small_SMD_Proto_Pad, Connectors:Small_SMD_Proto_Pad, B.Cu at (99.4, 76.5)
- added REF**: Small_SMD_Proto_Pad, Connectors:Small_SMD_Proto_Pad, B.Cu at (105.7, 71.4)
- added REF**: Small_SMD_Proto_Pad, Connectors:Small_SMD_Proto_Pad, B.Cu at (128.6, 85.4)
- added REF**: Small_SMD_Proto_Pad, Connectors:Small_SMD_Proto_Pad, B.Cu at (104.4, 63.8)
- added REF**: Small_SMD_Proto_Pad, Connectors:Small_SMD_Proto_Pad, B.Cu at (107.0, 98.1)
- added REF**: Small_SMD_Proto_Pad, Connectors:Small_SMD_Proto_Pad, B.Cu at (112.1, 104.4)
- added REF**: Small_SMD_Proto_Pad, Connectors:Small_SMD_Proto_Pad, B.Cu at (129.8, 86.7)
- added REF**: Small_SMD_Proto_Pad, Connectors:Small_SMD_Proto_Pad, B.Cu at (142.5, 87.9)
- added REF**: Small_SMD_Proto_Pad, Connectors:Small_SMD_Proto_Pad, B.Cu at (141.3, 86.7)
- added REF**: Small_SMD_Proto_Pad, Connectors:Small_SMD_Proto_Pad, F.Cu at (114.6, 100.6)
- added REF**: Small_SMD_Proto_Pad, Connectors:Small_SMD_Proto_Pad, B.Cu at (140.0, 93.0)
- added REF**: Small_SMD_Proto_Pad, Connectors:Small_SMD_Proto_Pad, B.Cu at (112.1, 105.7)
- added REF**: Small_SMD_Proto_Pad, Connectors:Small_SMD_Proto_Pad, B.Cu at (108.3, 72.7)
- added REF**: Small_SMD_Proto_Pad, Connectors:Small_SMD_Proto_Pad, B.Cu at (118.4, 104.4)
- added REF**: Small_SMD_Proto_Pad, Connectors:Small_SMD_Proto_Pad, B.Cu at (131.1, 96.8)
- added REF**: Small_SMD_Proto_Pad, Connectors:Small_SMD_Proto_Pad, B.Cu at (110.8, 104.4)
- added REF**: Small_SMD_Proto_Pad, Connectors:Small_SMD_Proto_Pad, B.Cu at (101.9, 68.9)
- added REF**: Small_SMD_Proto_Pad, Connectors:Small_SMD_Proto_Pad, B.Cu at (114.6, 99.4)
- added REF**: Small_SMD_Proto_Pad, Connectors:Small_SMD_Proto_Pad, B.Cu at (133.7, 84.1)
- added REF**: Small_SMD_Proto_Pad, Connectors:Small_SMD_Proto_Pad, B.Cu at (110.8, 103.2)
- added REF**: Small_SMD_Proto_Pad, Connectors:Small_SMD_Proto_Pad, F.Cu at (137.5, 93.0)
- added REF**: Small_SMD_Proto_Pad, Connectors:Small_SMD_Proto_Pad, B.Cu at (109.5, 90.5)
- added REF**: Small_SMD_Proto_Pad, Connectors:Small_SMD_Proto_Pad, B.Cu at (109.5, 74.0)
- added REF**: Small_SMD_Proto_Pad, Connectors:Small_SMD_Proto_Pad, B.Cu at (108.3, 71.4)
- added REF**: Small_SMD_Proto_Pad, Connectors:Small_SMD_Proto_Pad, B.Cu at (128.6, 100.6)
- added REF**: Small_SMD_Proto_Pad, Connectors:Small_SMD_Proto_Pad, B.Cu at (113.3, 65.1)
- added REF**: Small_SMD_Proto_Pad, Connectors:Small_SMD_Proto_Pad, B.Cu at (122.2, 87.9)
- added REF**: Small_SMD_Proto_Pad, Connectors:Small_SMD_Proto_Pad, B.Cu at (118.4, 107.0)
- added REF**: Small_SMD_Proto_Pad, Connectors:Small_SMD_Proto_Pad, B.Cu at (118.4, 105.7)
- added REF**: Small_SMD_Proto_Pad, Connectors:Small_SMD_Proto_Pad, B.Cu at (114.6, 85.4)
- added REF**: Small_SMD_Proto_Pad, Connectors:Small_SMD_Proto_Pad, B.Cu at (122.2, 98.1)
- added REF**: Small_SMD_Proto_Pad, Connectors:Small_SMD_Proto_Pad, F.Cu at (104.4, 99.4)
- added REF**: Small_SMD_Proto_Pad, Connectors:Small_SMD_Proto_Pad, B.Cu at (115.9, 74.0)
- added REF**: Small_SMD_Proto_Pad, Connectors:Small_SMD_Proto_Pad, B.Cu at (103.2, 81.6)
- added REF**: Small_SMD_Proto_Pad, Connectors:Small_SMD_Proto_Pad, B.Cu at (112.1, 70.2)
- added REF**: Small_SMD_Proto_Pad, Connectors:Small_SMD_Proto_Pad, B.Cu at (124.8, 95.6)
- added REF**: Small_SMD_Proto_Pad, Connectors:Small_SMD_Proto_Pad, B.Cu at (118.4, 82.9)
- added REF**: Small_SMD_Proto_Pad, Connectors:Small_SMD_Proto_Pad, B.Cu at (107.0, 104.4)
- added REF**: Small_SMD_Proto_Pad, Connectors:Small_SMD_Proto_Pad, B.Cu at (126.0, 86.7)
- added REF**: Small_SMD_Proto_Pad, Connectors:Small_SMD_Proto_Pad, B.Cu at (123.5, 103.2)
- added REF**: Small_SMD_Proto_Pad, Connectors:Small_SMD_Proto_Pad, B.Cu at (134.9, 93.0)
- added REF**: Small_SMD_Proto_Pad, Connectors:Small_SMD_Proto_Pad, B.Cu at (121.0, 98.1)
- added REF**: Small_SMD_Proto_Pad, Connectors:Small_SMD_Proto_Pad, F.Cu at (141.3, 89.2)
- added REF**: Small_SMD_Proto_Pad, Connectors:Small_SMD_Proto_Pad, B.Cu at (101.9, 85.4)
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Routing:
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- added copper zone on B.Cu, net GND
- added copper zone on F.Cu, net GND
Other:
- board text added: "+"
- board text added: "-"
- board text added: "1S LiPo"
- board text added: "A"
- board text added: "B"
- board text added: "CHG"
- board text added: "GND"
- board text added: "LED"
- board text added: "PA0"
- board text added: "PA1"
- board text added: "PA16"
- board text added: "PA17"
- board text added: "PA18"
- board text added: "PA19"
- board text added: "PA2"
- board text added: "PA23"
- board text added: "PA27"
- board text added: "PA28"
- board text added: "PA3"
- board text added: "PA6"
- board text added: "PA7"
- board text added: "PB2"
- board text added: "PB3"
- board text added: "PB9"
- board text added: "RESET"
- board text added: "RX"
- board text added: "SWDCLK"
- board text added: "SWDIO"
- board text added: "TX"
- board text added: "VCC"
- board text added: "VUSB"
- board text added: "X"
- board text added: "Y"
- board text added: "~RESET"
- board text removed: "@your_twitter_handle"

Commit message: gregdavill: Initial commit of new badge design
Parts:
- removed the R4 at (98.6, 118.0)
- removed REF** (x1161): Small_SMD_Proto_Pad, Connectors:Small_SMD_Proto_Pad
- removed REF** (x32): PTH_Proto_pad, Connectors:PTH_Proto_pad
- removed the TP1 at (77.1, 103.8)
- removed the U5 at (63.0, 131.4)
- added C13: 10uF, Capacitor_SMD:C_0603_1608Metric, F.Cu at (63.2, 141.0)
- added C14: 10uF, Capacitor_SMD:C_0603_1608Metric, F.Cu at (63.2, 139.5)
- added D100: LED, LED_SMD:LED_0402_1005Metric, F.Cu at (97.0, 70.7)
- added D101: LED, LED_SMD:LED_0402_1005Metric, F.Cu at (98.3, 72.0)
- added D102: LED, LED_SMD:LED_0402_1005Metric, F.Cu at (99.6, 73.3)
- added D103: LED, LED_SMD:LED_0402_1005Metric, F.Cu at (101.0, 74.6)
- added D104: LED, LED_SMD:LED_0402_1005Metric, F.Cu at (102.3, 75.9)
- added D105: LED, LED_SMD:LED_0402_1005Metric, F.Cu at (103.6, 77.2)
- added D106: LED, LED_SMD:LED_0402_1005Metric, F.Cu at (104.9, 78.5)
- added D107: LED, LED_SMD:LED_0402_1005Metric, F.Cu at (106.2, 79.8)
- added D108: LED, LED_SMD:LED_0402_1005Metric, F.Cu at (107.5, 81.1)
- added D109: LED, LED_SMD:LED_0402_1005Metric, F.Cu at (108.8, 82.4)
- added D110: LED, LED_SMD:LED_0402_1005Metric, F.Cu at (110.1, 83.7)
- added D111: LED, LED_SMD:LED_0402_1005Metric, F.Cu at (111.4, 85.0)
- added D112: LED, LED_SMD:LED_0402_1005Metric, F.Cu at (112.7, 86.3)
- added D113: LED, LED_SMD:LED_0402_1005Metric, F.Cu at (114.0, 87.6)
- added D114: LED, LED_SMD:LED_0402_1005Metric, F.Cu at (115.3, 88.9)
- added D115: LED, LED_SMD:LED_0402_1005Metric, F.Cu at (116.6, 90.2)
- added D116: LED, LED_SMD:LED_0402_1005Metric, F.Cu at (117.9, 91.5)
- added D117: LED, LED_SMD:LED_0402_1005Metric, F.Cu at (119.2, 92.8)
- added D118: LED, LED_SMD:LED_0402_1005Metric, F.Cu at (120.5, 94.1)
- added D119: LED, LED_SMD:LED_0402_1005Metric, F.Cu at (121.8, 95.4)
- added D120: LED, LED_SMD:LED_0402_1005Metric, F.Cu at (123.1, 96.7)
- added D121: LED, LED_SMD:LED_0402_1005Metric, F.Cu at (124.4, 98.0)
- added D122: LED, LED_SMD:LED_0402_1005Metric, F.Cu at (125.7, 99.3)
- added D123: LED, LED_SMD:LED_0402_1005Metric, F.Cu at (127.0, 100.6)
- added D124: LED, LED_SMD:LED_0402_1005Metric, F.Cu at (128.3, 101.9)
- added D125: LED, LED_SMD:LED_0402_1005Metric, F.Cu at (129.6, 103.2)
- added D126: LED, LED_SMD:LED_0402_1005Metric, F.Cu at (130.9, 104.5)
- added D127: LED, LED_SMD:LED_0402_1005Metric, F.Cu at (132.2, 105.8)
- added D128: LED, LED_SMD:LED_0402_1005Metric, F.Cu at (133.5, 107.1)
- added D129: LED, LED_SMD:LED_0402_1005Metric, F.Cu at (91.9, 68.3)
- added D130: LED, LED_SMD:LED_0402_1005Metric, F.Cu at (93.2, 69.6)
- added D131: LED, LED_SMD:LED_0402_1005Metric, F.Cu at (94.5, 70.9)
- added D132: LED, LED_SMD:LED_0402_1005Metric, F.Cu at (95.8, 72.2)
- added D133: LED, LED_SMD:LED_0402_1005Metric, F.Cu at (97.1, 73.5)
- added D134: LED, LED_SMD:LED_0402_1005Metric, F.Cu at (98.4, 74.8)
- added D135: LED, LED_SMD:LED_0402_1005Metric, F.Cu at (99.6, 76.1)
- added D136: LED, LED_SMD:LED_0402_1005Metric, F.Cu at (100.9, 77.4)
- added D137: LED, LED_SMD:LED_0402_1005Metric, F.Cu at (102.2, 78.7)
- added D138: LED, LED_SMD:LED_0402_1005Metric, F.Cu at (103.5, 80.0)
- added D139: LED, LED_SMD:LED_0402_1005Metric, F.Cu at (104.8, 81.2)
- added D140: LED, LED_SMD:LED_0402_1005Metric, F.Cu at (106.1, 82.5)
- added D141: LED, LED_SMD:LED_0402_1005Metric, F.Cu at (107.4, 83.8)
- added D142: LED, LED_SMD:LED_0402_1005Metric, F.Cu at (108.7, 85.1)
- added D143: LED, LED_SMD:LED_0402_1005Metric, F.Cu at (110.0, 86.4)
- added D144: LED, LED_SMD:LED_0402_1005Metric, F.Cu at (111.3, 87.7)
- added D145: LED, LED_SMD:LED_0402_1005Metric, F.Cu at (112.5, 89.0)
- added D146: LED, LED_SMD:LED_0402_1005Metric, F.Cu at (113.8, 90.3)
- added D147: LED, LED_SMD:LED_0402_1005Metric, F.Cu at (115.1, 91.6)
- added D148: LED, LED_SMD:LED_0402_1005Metric, F.Cu at (116.4, 92.9)
- added D149: LED, LED_SMD:LED_0402_1005Metric, F.Cu at (117.7, 94.1)
- added D150: LED, LED_SMD:LED_0402_1005Metric, F.Cu at (119.0, 95.4)
- added D151: LED, LED_SMD:LED_0402_1005Metric, F.Cu at (120.3, 96.7)
- added D152: LED, LED_SMD:LED_0402_1005Metric, F.Cu at (121.6, 98.0)
- added D153: LED, LED_SMD:LED_0402_1005Metric, F.Cu at (122.9, 99.3)
- added D154: LED, LED_SMD:LED_0402_1005Metric, F.Cu at (124.1, 100.6)
- added D155: LED, LED_SMD:LED_0402_1005Metric, F.Cu at (125.4, 101.9)
- added D156: LED, LED_SMD:LED_0402_1005Metric, F.Cu at (126.7, 103.2)
- added D157: LED, LED_SMD:LED_0402_1005Metric, F.Cu at (128.0, 104.5)
- added D158: LED, LED_SMD:LED_0402_1005Metric, F.Cu at (129.3, 105.8)
- added D159: LED, LED_SMD:LED_0402_1005Metric, F.Cu at (130.6, 107.0)
- added D160: LED, LED_SMD:LED_0402_1005Metric, F.Cu at (131.9, 108.3)
- added D161: LED, LED_SMD:LED_0402_1005Metric, F.Cu at (90.6, 69.9)
- added D162: LED, LED_SMD:LED_0402_1005Metric, F.Cu at (91.9, 71.2)
- added D163: LED, LED_SMD:LED_0402_1005Metric, F.Cu at (93.2, 72.5)
- added D164: LED, LED_SMD:LED_0402_1005Metric, F.Cu at (94.5, 73.8)
- added D165: LED, LED_SMD:LED_0402_1005Metric, F.Cu at (95.8, 75.0)
- added D166: LED, LED_SMD:LED_0402_1005Metric, F.Cu at (97.0, 76.3)
- added D167: LED, LED_SMD:LED_0402_1005Metric, F.Cu at (98.3, 77.6)
- added D168: LED, LED_SMD:LED_0402_1005Metric, F.Cu at (99.6, 78.9)
- added D169: LED, LED_SMD:LED_0402_1005Metric, F.Cu at (100.9, 80.2)
- added D170: LED, LED_SMD:LED_0402_1005Metric, F.Cu at (102.2, 81.4)
- added D171: LED, LED_SMD:LED_0402_1005Metric, F.Cu at (103.4, 82.7)
- added D172: LED, LED_SMD:LED_0402_1005Metric, F.Cu at (104.7, 84.0)
- added D173: LED, LED_SMD:LED_0402_1005Metric, F.Cu at (106.0, 85.3)
- added D174: LED, LED_SMD:LED_0402_1005Metric, F.Cu at (107.3, 86.6)
- added D175: LED, LED_SMD:LED_0402_1005Metric, F.Cu at (108.6, 87.8)
- added D176: LED, LED_SMD:LED_0402_1005Metric, F.Cu at (109.8, 89.1)
- added D177: LED, LED_SMD:LED_0402_1005Metric, F.Cu at (111.1, 90.4)
- added D178: LED, LED_SMD:LED_0402_1005Metric, F.Cu at (112.4, 91.7)
- added D179: LED, LED_SMD:LED_0402_1005Metric, F.Cu at (113.7, 93.0)
- added D180: LED, LED_SMD:LED_0402_1005Metric, F.Cu at (115.0, 94.2)
- added D181: LED, LED_SMD:LED_0402_1005Metric, F.Cu at (116.2, 95.5)
- added D182: LED, LED_SMD:LED_0402_1005Metric, F.Cu at (117.5, 96.8)
- added D183: LED, LED_SMD:LED_0402_1005Metric, F.Cu at (118.8, 98.1)
- added D184: LED, LED_SMD:LED_0402_1005Metric, F.Cu at (120.1, 99.4)
- added D185: LED, LED_SMD:LED_0402_1005Metric, F.Cu at (121.4, 100.6)
- added D186: LED, LED_SMD:LED_0402_1005Metric, F.Cu at (122.6, 101.9)
- added D187: LED, LED_SMD:LED_0402_1005Metric, F.Cu at (123.9, 103.2)
- added D188: LED, LED_SMD:LED_0402_1005Metric, F.Cu at (125.2, 104.5)
- added D189: LED, LED_SMD:LED_0402_1005Metric, F.Cu at (126.5, 105.8)
- added D190: LED, LED_SMD:LED_0402_1005Metric, F.Cu at (127.8, 107.0)
- added D191: LED, LED_SMD:LED_0402_1005Metric, F.Cu at (129.0, 108.3)
- added D192: LED, LED_SMD:LED_0402_1005Metric, F.Cu at (130.3, 109.6)
- added D193: LED, LED_SMD:LED_0402_1005Metric, F.Cu at (89.4, 71.5)
- added D194: LED, LED_SMD:LED_0402_1005Metric, F.Cu at (90.6, 72.7)
- added D195: LED, LED_SMD:LED_0402_1005Metric, F.Cu at (91.9, 74.0)
- added D196: LED, LED_SMD:LED_0402_1005Metric, F.Cu at (93.2, 75.3)
- added D197: LED, LED_SMD:LED_0402_1005Metric, F.Cu at (94.4, 76.5)
- added D198: LED, LED_SMD:LED_0402_1005Metric, F.Cu at (95.7, 77.8)
- added D199: LED, LED_SMD:LED_0402_1005Metric, F.Cu at (97.0, 79.1)
- added D200: LED, LED_SMD:LED_0402_1005Metric, F.Cu at (98.3, 80.4)
- added D201: LED, LED_SMD:LED_0402_1005Metric, F.Cu at (99.5, 81.6)
- added D202: LED, LED_SMD:LED_0402_1005Metric, F.Cu at (100.8, 82.9)
- added D203: LED, LED_SMD:LED_0402_1005Metric, F.Cu at (102.1, 84.2)
- added D204: LED, LED_SMD:LED_0402_1005Metric, F.Cu at (103.3, 85.4)
- added D205: LED, LED_SMD:LED_0402_1005Metric, F.Cu at (104.6, 86.7)
- added D206: LED, LED_SMD:LED_0402_1005Metric, F.Cu at (105.9, 88.0)
- added D207: LED, LED_SMD:LED_0402_1005Metric, F.Cu at (107.2, 89.3)
- added D208: LED, LED_SMD:LED_0402_1005Metric, F.Cu at (108.4, 90.5)
- added D209: LED, LED_SMD:LED_0402_1005Metric, F.Cu at (109.7, 91.8)
- added D210: LED, LED_SMD:LED_0402_1005Metric, F.Cu at (111.0, 93.1)
- added D211: LED, LED_SMD:LED_0402_1005Metric, F.Cu at (112.2, 94.3)
- added D212: LED, LED_SMD:LED_0402_1005Metric, F.Cu at (113.5, 95.6)
- added D213: LED, LED_SMD:LED_0402_1005Metric, F.Cu at (114.8, 96.9)
- added D214: LED, LED_SMD:LED_0402_1005Metric, F.Cu at (116.1, 98.2)
- added D215: LED, LED_SMD:LED_0402_1005Metric, F.Cu at (117.3, 99.4)
- added D216: LED, LED_SMD:LED_0402_1005Metric, F.Cu at (118.6, 100.7)
- added D217: LED, LED_SMD:LED_0402_1005Metric, F.Cu at (119.9, 102.0)
- added D218: LED, LED_SMD:LED_0402_1005Metric, F.Cu at (121.1, 103.2)
- added D219: LED, LED_SMD:LED_0402_1005Metric, F.Cu at (122.4, 104.5)
- added D220: LED, LED_SMD:LED_0402_1005Metric, F.Cu at (123.7, 105.8)
- added D221: LED, LED_SMD:LED_0402_1005Metric, F.Cu at (125.0, 107.1)
- added D222: LED, LED_SMD:LED_0402_1005Metric, F.Cu at (126.2, 108.3)
- added D223: LED, LED_SMD:LED_0402_1005Metric, F.Cu at (127.5, 109.6)
- added D224: LED, LED_SMD:LED_0402_1005Metric, F.Cu at (128.8, 110.9)
- added D225: LED, LED_SMD:LED_0402_1005Metric, F.Cu at (88.1, 73.0)
- added D226: LED, LED_SMD:LED_0402_1005Metric, F.Cu at (89.3, 74.3)
- added D227: LED, LED_SMD:LED_0402_1005Metric, F.Cu at (90.6, 75.5)
- added D228: LED, LED_SMD:LED_0402_1005Metric, F.Cu at (91.9, 76.8)
- added D229: LED, LED_SMD:LED_0402_1005Metric, F.Cu at (93.1, 78.1)
- added D230: LED, LED_SMD:LED_0402_1005Metric, F.Cu at (94.4, 79.3)
- added D231: LED, LED_SMD:LED_0402_1005Metric, F.Cu at (95.6, 80.6)
- added D232: LED, LED_SMD:LED_0402_1005Metric, F.Cu at (96.9, 81.8)
- added D233: LED, LED_SMD:LED_0402_1005Metric, F.Cu at (98.2, 83.1)
- added D234: LED, LED_SMD:LED_0402_1005Metric, F.Cu at (99.4, 84.4)
- added D235: LED, LED_SMD:LED_0402_1005Metric, F.Cu at (100.7, 85.6)
- added D236: LED, LED_SMD:LED_0402_1005Metric, F.Cu at (102.0, 86.9)
- added D237: LED, LED_SMD:LED_0402_1005Metric, F.Cu at (103.2, 88.2)
- added D238: LED, LED_SMD:LED_0402_1005Metric, F.Cu at (104.5, 89.4)
- added D239: LED, LED_SMD:LED_0402_1005Metric, F.Cu at (105.8, 90.7)
- added D240: LED, LED_SMD:LED_0402_1005Metric, F.Cu at (107.0, 92.0)
- added D241: LED, LED_SMD:LED_0402_1005Metric, F.Cu at (108.3, 93.2)
- added D242: LED, LED_SMD:LED_0402_1005Metric, F.Cu at (109.5, 94.5)
- added D243: LED, LED_SMD:LED_0402_1005Metric, F.Cu at (110.8, 95.7)
- added D244: LED, LED_SMD:LED_0402_1005Metric, F.Cu at (112.1, 97.0)
- added D245: LED, LED_SMD:LED_0402_1005Metric, F.Cu at (113.3, 98.3)
- added D246: LED, LED_SMD:LED_0402_1005Metric, F.Cu at (114.6, 99.5)
- added D247: LED, LED_SMD:LED_0402_1005Metric, F.Cu at (115.9, 100.8)
- added D248: LED, LED_SMD:LED_0402_1005Metric, F.Cu at (117.1, 102.1)
- added D249: LED, LED_SMD:LED_0402_1005Metric, F.Cu at (118.4, 103.3)
- added D25: LED, LED_SMD:LED_0402_1005Metric, F.Cu at (129.0, 94.1)
- added D250: LED, LED_SMD:LED_0402_1005Metric, F.Cu at (119.7, 104.6)
- added D251: LED, LED_SMD:LED_0402_1005Metric, F.Cu at (120.9, 105.9)
- added D252: LED, LED_SMD:LED_0402_1005Metric, F.Cu at (122.2, 107.1)
- added D253: LED, LED_SMD:LED_0402_1005Metric, F.Cu at (123.4, 108.4)
- added D254: LED, LED_SMD:LED_0402_1005Metric, F.Cu at (124.7, 109.6)
- added D255: LED, LED_SMD:LED_0402_1005Metric, F.Cu at (126.0, 110.9)
- added D256: LED, LED_SMD:LED_0402_1005Metric, F.Cu at (127.2, 112.2)
- added D257: LED, LED_SMD:LED_0402_1005Metric, F.Cu at (86.8, 74.5)
- added D258: LED, LED_SMD:LED_0402_1005Metric, F.Cu at (88.0, 75.8)
- added D259: LED, LED_SMD:LED_0402_1005Metric, F.Cu at (89.3, 77.0)
- added D26: LED, LED_SMD:LED_0402_1005Metric, F.Cu at (130.3, 95.4)
- added D260: LED, LED_SMD:LED_0402_1005Metric, F.Cu at (90.5, 78.3)
- added D261: LED, LED_SMD:LED_0402_1005Metric, F.Cu at (91.8, 79.5)
- added D262: LED, LED_SMD:LED_0402_1005Metric, F.Cu at (93.0, 80.8)
- added D263: LED, LED_SMD:LED_0402_1005Metric, F.Cu at (94.3, 82.1)
- added D264: LED, LED_SMD:LED_0402_1005Metric, F.Cu at (95.6, 83.3)
- added D265: LED, LED_SMD:LED_0402_1005Metric, F.Cu at (96.8, 84.6)
- added D266: LED, LED_SMD:LED_0402_1005Metric, F.Cu at (98.1, 85.8)
- added D267: LED, LED_SMD:LED_0402_1005Metric, F.Cu at (99.3, 87.1)
- added D268: LED, LED_SMD:LED_0402_1005Metric, F.Cu at (100.6, 88.3)
- added D269: LED, LED_SMD:LED_0402_1005Metric, F.Cu at (101.8, 89.6)
- added D27: LED, LED_SMD:LED_0402_1005Metric, F.Cu at (131.6, 96.8)
- added D270: LED, LED_SMD:LED_0402_1005Metric, F.Cu at (103.1, 90.9)
- added D271: LED, LED_SMD:LED_0402_1005Metric, F.Cu at (104.4, 92.1)
- added D272: LED, LED_SMD:LED_0402_1005Metric, F.Cu at (105.6, 93.4)
- added D273: LED, LED_SMD:LED_0402_1005Metric, F.Cu at (106.9, 94.6)
- added D274: LED, LED_SMD:LED_0402_1005Metric, F.Cu at (108.1, 95.9)
- added D275: LED, LED_SMD:LED_0402_1005Metric, F.Cu at (109.4, 97.1)
- added D276: LED, LED_SMD:LED_0402_1005Metric, F.Cu at (110.6, 98.4)
- added D277: LED, LED_SMD:LED_0402_1005Metric, F.Cu at (111.9, 99.7)
- added D278: LED, LED_SMD:LED_0402_1005Metric, F.Cu at (113.2, 100.9)
- added D279: LED, LED_SMD:LED_0402_1005Metric, F.Cu at (114.4, 102.2)
- added D28: LED, LED_SMD:LED_0402_1005Metric, F.Cu at (133.0, 98.1)
- added D280: LED, LED_SMD:LED_0402_1005Metric, F.Cu at (115.7, 103.4)
- added D281: LED, LED_SMD:LED_0402_1005Metric, F.Cu at (116.9, 104.7)
- added D282: LED, LED_SMD:LED_0402_1005Metric, F.Cu at (118.2, 105.9)
- added D283: LED, LED_SMD:LED_0402_1005Metric, F.Cu at (119.4, 107.2)
- added D284: LED, LED_SMD:LED_0402_1005Metric, F.Cu at (120.7, 108.5)
- added D285: LED, LED_SMD:LED_0402_1005Metric, F.Cu at (122.0, 109.7)
- added D286: LED, LED_SMD:LED_0402_1005Metric, F.Cu at (123.2, 111.0)
- added D287: LED, LED_SMD:LED_0402_1005Metric, F.Cu at (124.5, 112.2)
- added D288: LED, LED_SMD:LED_0402_1005Metric, F.Cu at (125.7, 113.5)
- added D289: LED, LED_SMD:LED_0402_1005Metric, F.Cu at (85.4, 76.0)
- added D29: LED, LED_SMD:LED_0402_1005Metric, F.Cu at (134.3, 99.5)
- added D290: LED, LED_SMD:LED_0402_1005Metric, F.Cu at (86.7, 77.3)
- added D291: LED, LED_SMD:LED_0402_1005Metric, F.Cu at (87.9, 78.5)
- added D292: LED, LED_SMD:LED_0402_1005Metric, F.Cu at (89.2, 79.8)
- added D293: LED, LED_SMD:LED_0402_1005Metric, F.Cu at (90.4, 81.0)
- added D294: LED, LED_SMD:LED_0402_1005Metric, F.Cu at (91.7, 82.3)
- added D295: LED, LED_SMD:LED_0402_1005Metric, F.Cu at (92.9, 83.5)
- added D296: LED, LED_SMD:LED_0402_1005Metric, F.Cu at (94.2, 84.8)
- added D297: LED, LED_SMD:LED_0402_1005Metric, F.Cu at (95.4, 86.0)
- added D298: LED, LED_SMD:LED_0402_1005Metric, F.Cu at (96.7, 87.3)
- added D299: LED, LED_SMD:LED_0402_1005Metric, F.Cu at (97.9, 88.5)
- added D30: LED, LED_SMD:LED_0402_1005Metric, F.Cu at (135.7, 100.8)
- added D300: LED, LED_SMD:LED_0402_1005Metric, F.Cu at (99.2, 89.8)
- added D301: LED, LED_SMD:LED_0402_1005Metric, F.Cu at (100.4, 91.0)
- added D302: LED, LED_SMD:LED_0402_1005Metric, F.Cu at (101.7, 92.3)
- added D303: LED, LED_SMD:LED_0402_1005Metric, F.Cu at (102.9, 93.5)
- added D304: LED, LED_SMD:LED_0402_1005Metric, F.Cu at (104.2, 94.8)
- added D305: LED, LED_SMD:LED_0402_1005Metric, F.Cu at (105.5, 96.0)
- added D306: LED, LED_SMD:LED_0402_1005Metric, F.Cu at (106.7, 97.3)
- added D307: LED, LED_SMD:LED_0402_1005Metric, F.Cu at (108.0, 98.5)
- added D308: LED, LED_SMD:LED_0402_1005Metric, F.Cu at (109.2, 99.8)
- added D309: LED, LED_SMD:LED_0402_1005Metric, F.Cu at (110.5, 101.0)
- added D31: LED, LED_SMD:LED_0402_1005Metric, F.Cu at (137.0, 102.1)
- added D310: LED, LED_SMD:LED_0402_1005Metric, F.Cu at (111.7, 102.3)
- added D311: LED, LED_SMD:LED_0402_1005Metric, F.Cu at (113.0, 103.5)
- added D312: LED, LED_SMD:LED_0402_1005Metric, F.Cu at (114.2, 104.8)
- added D313: LED, LED_SMD:LED_0402_1005Metric, F.Cu at (115.5, 106.1)
- added D314: LED, LED_SMD:LED_0402_1005Metric, F.Cu at (116.7, 107.3)
- added D315: LED, LED_SMD:LED_0402_1005Metric, F.Cu at (118.0, 108.6)
- added D316: LED, LED_SMD:LED_0402_1005Metric, F.Cu at (119.2, 109.8)
- added D317: LED, LED_SMD:LED_0402_1005Metric, F.Cu at (120.5, 111.1)
- added D318: LED, LED_SMD:LED_0402_1005Metric, F.Cu at (121.7, 112.3)
- added D319: LED, LED_SMD:LED_0402_1005Metric, F.Cu at (123.0, 113.6)
- added D32: LED, LED_SMD:LED_0402_1005Metric, F.Cu at (138.3, 103.5)
- added D320: LED, LED_SMD:LED_0402_1005Metric, F.Cu at (124.2, 114.8)
- added D321: LED, LED_SMD:LED_0402_1005Metric, F.Cu at (84.1, 77.5)
- added D322: LED, LED_SMD:LED_0402_1005Metric, F.Cu at (85.3, 78.7)
- added D323: LED, LED_SMD:LED_0402_1005Metric, F.Cu at (86.6, 80.0)
- added D324: LED, LED_SMD:LED_0402_1005Metric, F.Cu at (87.8, 81.2)
- added D325: LED, LED_SMD:LED_0402_1005Metric, F.Cu at (89.1, 82.5)
- added D326: LED, LED_SMD:LED_0402_1005Metric, F.Cu at (90.3, 83.7)
- added D327: LED, LED_SMD:LED_0402_1005Metric, F.Cu at (91.6, 85.0)
- added D328: LED, LED_SMD:LED_0402_1005Metric, F.Cu at (92.8, 86.2)
- added D329: LED, LED_SMD:LED_0402_1005Metric, F.Cu at (94.1, 87.5)
- added D33: LED, LED_SMD:LED_0402_1005Metric, F.Cu at (95.6, 63.5)
- added D330: LED, LED_SMD:LED_0402_1005Metric, F.Cu at (95.3, 88.7)
- added D331: LED, LED_SMD:LED_0402_1005Metric, F.Cu at (96.5, 90.0)
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- renumbered D25 to D513, D26 to D514, R12 to R10, R13 to R11, R14 to R12, R15 to R13, R16 to R14, R17 to R15, R18 to R16, R5 to R3, R6 to R4, R7 to R5, R8 to R6, R9 to R7, R10 to R8, TP17 to TP1, TP8 to TP10, TP9 to TP11, TP10 to TP12, TP11 to TP13, TP12 to TP14, TP18 to TP2, TP2 to TP4, TP3 to TP5, TP4 to TP6, TP5 to TP7, TP6 to TP8, TP7 to TP9, U3 to U5, U4 to U6, U6 to U8, U7 to U9
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Connections:
- C10 pad 1: VCC -> Net-(C10-Pad1)
- C10 pad 2: GND -> VCC
- C9 pad 1: /1s LiPo/BATT_PLUS -> GND
- C9 pad 2: GND -> /1s LiPo/BATT_PLUS
- D1 pad 1: VCC -> COL_GA0
- D1 pad 2: Net-(D1-Pad2) -> /ISSI 12 RGB A/COM_6
- D10 pad 1: VCC -> COL_GA9
- D10 pad 2: Net-(D10-Pad2) -> /ISSI 12 RGB A/COM_6
- D11 pad 1: VCC -> COL_GA10
- D11 pad 2: Net-(D11-Pad2) -> /ISSI 12 RGB A/COM_6
- D12 pad 1: VCC -> COL_GA11
- D12 pad 2: Net-(D12-Pad2) -> /ISSI 12 RGB A/COM_6
- D13 pad 1: VCC -> COL_GA12
- D13 pad 2: Net-(D13-Pad2) -> /ISSI 12 RGB A/COM_6
- D14 pad 1: VCC -> COL_GA13
- D14 pad 2: Net-(D14-Pad2) -> /ISSI 12 RGB A/COM_6
- D15 pad 1: VCC -> COL_GA14
- D15 pad 2: Net-(D15-Pad2) -> /ISSI 12 RGB A/COM_6
- D16 pad 1: VCC -> COL_GA15
- D16 pad 2: Net-(D16-Pad2) -> /ISSI 12 RGB A/COM_6
- D17 pad 1: VCC -> COL_GA16
- D17 pad 2: Net-(D17-Pad2) -> /ISSI 12 RGB A/COM_6
- D18 pad 1: VCC -> COL_GA17
- D18 pad 2: Net-(D18-Pad2) -> /ISSI 12 RGB A/COM_6
- D19 pad 1: VCC -> COL_GA18
- D19 pad 2: Net-(D19-Pad2) -> /ISSI 12 RGB A/COM_6
- D2 pad 1: VCC -> COL_GA1
- D2 pad 2: Net-(D2-Pad2) -> /ISSI 12 RGB A/COM_6
- D20 pad 1: VCC -> COL_GA19
- D20 pad 2: Net-(D20-Pad2) -> /ISSI 12 RGB A/COM_6
- D21 pad 1: VCC -> COL_GA20
- D21 pad 2: Net-(D21-Pad2) -> /ISSI 12 RGB A/COM_6
- D22 pad 1: VCC -> COL_GA21
- D22 pad 2: Net-(D22-Pad2) -> /ISSI 12 RGB A/COM_6
- D23 pad 1: VCC -> COL_GA22
- D23 pad 2: Net-(D23-Pad2) -> /ISSI 12 RGB A/COM_6
- D24 pad 1: VCC -> COL_GA23
- D24 pad 2: Net-(D24-Pad2) -> /ISSI 12 RGB A/COM_6
- D3 pad 1: VCC -> COL_GA2
- D3 pad 2: Net-(D3-Pad2) -> /ISSI 12 RGB A/COM_6
- D4 pad 1: VCC -> COL_GA3
- D4 pad 2: Net-(D4-Pad2) -> /ISSI 12 RGB A/COM_6
- D5 pad 1: VCC -> COL_GA4
- D5 pad 2: Net-(D5-Pad2) -> /ISSI 12 RGB A/COM_6
- D6 pad 1: VCC -> COL_GA5
- D6 pad 2: Net-(D6-Pad2) -> /ISSI 12 RGB A/COM_6
- D7 pad 1: VCC -> COL_GA6
- D7 pad 2: Net-(D7-Pad2) -> /ISSI 12 RGB A/COM_6
- D8 pad 1: VCC -> COL_GA7
- D8 pad 2: Net-(D8-Pad2) -> /ISSI 12 RGB A/COM_6
- D9 pad 1: VCC -> COL_GA8
- D9 pad 2: Net-(D9-Pad2) -> /ISSI 12 RGB A/COM_6
- IC1 pad 25: Net-(IC1-Pad25) -> /LED_BLANK
- IC1 pad 26: Net-(IC1-Pad26) -> /LED_LATCH
- IC1 pad 27: Net-(IC1-Pad27) -> /LED_SCLK
- IC1 pad 28: Net-(IC1-Pad28) -> /LED_DAT
- IC1 pad 37: /SDB -> (no net)
- R9 pad 1: GND -> VCC
- R9 pad 2: /SDB -> /LED_BLANK
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Routing:
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- added copper zone on In2.Cu, net GND
- added copper zone on In1.Cu, net VCC
- removed copper zone on B.Cu, net GND
- removed copper zone on F.Cu, net GND
Other:
- copper layers 2 -> 4
- board text added: "@gregdavill"
- board text added: "BLK"
- board text added: "CLK"
- board text added: "DAT"
- board text added: "LE"
- board text removed: "PA16"
- board text removed: "PA17"
- board text removed: "PA18"
- board text removed: "PA19"
