File: badge.kicad_sch (KiCad schematic)
At the start: 0 parts

Commit message: Added schematic, board and gerbers for my fork
Signed-off-by: Thomas Flummer <tf@flummer.net>
Parts:
- added SW1: A, Buttons:SW_SPST_TS3625A-HT, symbol Switch:SW_SPST
- added SW2: B, Buttons:SW_SPST_TS3625A-HT, symbol Switch:SW_SPST
- added SW3: X, Buttons:SW_SPST_TS3625A-HT, symbol Switch:SW_SPST
- added SW4: Y, Buttons:SW_SPST_TS3625A-HT, symbol Switch:SW_SPST
- added TP17: RX, Connectors:TestPoint_Large, symbol Connector:TestPoint
- added TP18: TX, Connectors:TestPoint_Large, symbol Connector:TestPoint
- added X1: #badgelife, badgelife_sao_v169bis:Badgelife-SAOv169-BADGE-2x3, symbol badgelife_shitty_addon_v169bis:Badgelife_sao_connector_v169bis
Connections:
- new net GND: SW1.2 (B), SW2.2 (B), SW3.2 (B), SW4.2 (B), X1.2 (GND)
- new net GPIO1: X1.5 (GPIO1)
- new net GPIO2: X1.6 (GPIO2)
- new net SAMD21/BTN_A: SW1.1 (A)
- new net SAMD21/BTN_B: SW2.1 (A)
- new net SAMD21/BTN_X: SW3.1 (A)
- new net SAMD21/BTN_Y: SW4.1 (A)
- new net SAMD21/UART_RX: TP17.1
- new net SAMD21/UART_TX: TP18.1
- new net SCL: X1.4 (SCL)
- new net SDA: X1.3 (SDA)
- new net VCC: X1.1 (VCC)
Other:
- added sheet 1s LiPo (1s_lipo.kicad_sch)
- added sheet ISSI 12 RGB A (issi_12_rgb.kicad_sch)
- added sheet ISSI 12 RGB B (issi_12_rgb.kicad_sch)
- added sheet SAMD21 (samd21.kicad_sch)
- title: KiCon 2020 Virtual Edition DIY Badge -> KiCon 2020 Virtual Edition Badge by Thomas Flummer

Commit message: gregdavill: Initial commit of new badge design
Parts:
- renumbered TP17 to TP1, TP18 to TP2
Other:
- removed sheet ISSI 12 RGB B
- sheet ISSI 12 RGB A ports: added BLANK, DAT, LATCH, SCLK; removed AD, SCL, SDA, SDB
- sheet SAMD21 ports: added LED_BLANK, LED_DAT, LED_LATCH, LED_SCLK; removed SDB

Commit message: add BOM
Parts:
- SW1, SW2, SW3, SW4: footprint Buttons:SW_SPST_TS3625A-HT -> Button_Switch_SMD:SW_SPST_PTS810; Mfg (none) -> C&K; PN (none) -> PTS810SJK250SMTRLFS
Changed lines of the file:
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@@
     (property "Reference" "SW1" (id 0) (at 151.13 133.35 0))
     (property "Value" "A" (id 1) (at 151.13 135.89 0))
-    (property "Footprint" "Buttons:SW_SPST_TS3625A-HT" (id 2) (at 151.13 139.7 0)
+    (property "Footprint" "Button_Switch_SMD:SW_SPST_PTS810" (id 2) (at 151.13 139.7 0)
       (effects (font (size 1.27 1.27)) hide)
     )
     (property "Datasheet" "~" (id 3) (at 151.13 139.7 0)
+      (effects (font (size 1.27 1.27)) hide)
+    )
+    (property "Mfg" "C&K" (id 4) (at 151.13 139.7 0)
+      (effects (font (size 1.27 1.27)) hide)
+    )
+    (property "PN" "PTS810SJK250SMTRLFS" (id 5) (at 151.13 139.7 0)
       (effects (font (size 1.27 1.27)) hide)
     )
@@
     (property "Reference" "SW2" (id 0) (at 151.13 143.51 0))
     (property "Value" "B" (id 1) (at 151.13 146.05 0))
-    (property "Footprint" "Buttons:SW_SPST_TS3625A-HT" (id 2) (at 151.13 149.86 0)
+    (property "Footprint" "Button_Switch_SMD:SW_SPST_PTS810" (id 2) (at 151.13 149.86 0)
       (effects (font (size 1.27 1.27)) hide)
     )
     (property "Datasheet" "~" (id 3) (at 151.13 149.86 0)
+      (effects (font (size 1.27 1.27)) hide)
+    )
+    (property "Mfg" "C&K" (id 4) (at 151.13 149.86 0)
+      (effects (font (size 1.27 1.27)) hide)
+    )
+    (property "PN" "PTS810SJK250SMTRLFS" (id 5) (at 151.13 149.86 0)
       (effects (font (size 1.27 1.27)) hide)
     )
@@
     (property "Reference" "SW3" (id 0) (at 151.13 153.67 0))
     (property "Value" "X" (id 1) (at 151.13 156.21 0))
-    (property "Footprint" "Buttons:SW_SPST_TS3625A-HT" (id 2) (at 151.13 160.02 0)
+    (property "Footprint" "Button_Switch_SMD:SW_SPST_PTS810" (id 2) (at 151.13 160.02 0)
       (effects (font (size 1.27 1.27)) hide)
     )
     (property "Datasheet" "~" (id 3) (at 151.13 160.02 0)
+      (effects (font (size 1.27 1.27)) hide)
+    )
+    (property "Mfg" "C&K" (id 4) (at 151.13 160.02 0)
+      (effects (font (size 1.27 1.27)) hide)
+    )
+    (property "PN" "PTS810SJK250SMTRLFS" (id 5) (at 151.13 160.02 0)
       (effects (font (size 1.27 1.27)) hide)
     )
@@
     (property "Reference" "SW4" (id 0) (at 151.13 163.83 0))
     (property "Value" "Y" (id 1) (at 151.13 166.37 0))
-    (property "Footprint" "Buttons:SW_SPST_TS3625A-HT" (id 2) (at 151.13 170.18 0)
+    (property "Footprint" "Button_Switch_SMD:SW_SPST_PTS810" (id 2) (at 151.13 170.18 0)
       (effects (font (size 1.27 1.27)) hide)
     )
@@
       (effects (font (size 1.27 1.27)) hide)
     )
+    (property "Mfg" "C&K" (id 4) (at 151.13 170.18 0)
+      (effects (font (size 1.27 1.27)) hide)
+    )
+    (property "PN" "PTS810SJK250SMTRLFS" (id 5) (at 151.13 170.18 0)
+      (effects (font (size 1.27 1.27)) hide)
+    )
