File: ledStripe.kicad_sch (KiCad schematic)
At the start: 32 parts

Commit message: add BOM
Parts:
- D481, D482, D483, D484, D485, D486, D487, D488, D489, D490, D491, D492, D493, D494, D495, D496, D497, D498, D499, D500, D501, D502, D503, D504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: Mfg (none) -> Foshan NationStar Optoelectronics; PN (none) -> NCD0402O1
